File: main.kicad_sch (KiCad schematic)
At the start: 45 parts, among them J1 MTA02-156, J2 MTA02-156, J3 MTA02-156, J4 MTA02-156, J5 MTA02-156, J6 MTA02-156, J7 MTA02-156

Commit message: Renamed footprints in libs to deal with error of importing to pcbdoc
Parts:
- V1, V2: footprint main:NOVAL -> main:TUBE
Changed lines of the file:
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@@
 			)
 		)
-		(property "Footprint" "main:NOVAL"
+		(property "Footprint" "main:TUBE"
 			(at 236.22 73.66 0)
 			(effects
@@
 			)
 		)
-		(property "Footprint" "main:NOVAL"
+		(property "Footprint" "main:TUBE"
 			(at 284.48 73.66 0)
 			(effects
@@
 			)
 		)
-		(property "Footprint" "main:NOVAL"
+		(property "Footprint" "main:TUBE"
 			(at 83.82 63.5 0)
 			(effects
@@
 			)
 		)
-		(property "Footprint" "main:NOVAL"
+		(property "Footprint" "main:TUBE"
 			(at 185.42 160.02 0)
 			(effects
@@
 			)
 		)
-		(property "Footprint" "main:NOVAL"
+		(property "Footprint" "main:TUBE"
 			(at 83.82 160.02 0)
 			(effects
@@
 			)
 		)
-		(property "Footprint" "main:NOVAL"
+		(property "Footprint" "main:TUBE"
 			(at 185.42 63.5 0)
 			(effects
